File: Senior Board File/SensorBoardR1.brd (EAGLE design)
At the start: 29.2 x 34 mm, 12 parts, among them T1 BC846, T2 BC846, T3 BC846

Commit message: 100% Build and Ready for R1 Purchase
Fixed a single wire that was needed
Parts:
- moved OPT3001 5.08 mm to (14.0, 17.8), turned to 270 degrees
Routing:
- net SDA: track 22.2 -> 48.0 mm, vias 0 -> 2
- net GND: track 51.3 -> 35.3 mm, vias 0 -> 1
- net INT: track 25.7 -> 28.8 mm, vias 2 -> 1
- net +3V3: track 88.1 -> 85.7 mm
- net SCL: track 30.1 -> 31.1 mm, vias 1 -> 0
